Commit message: Added CADI 1-2-3

File: docker_ws/py_pubsub/urdf/mapa1.xacro (robot description, xacro)
@@ -2,5 +2,5 @@
 <robot name="mapa_1" xmlns:xacro="http://www.ros.org/wiki/xacro">
 <!-- Introducir meshes -->
-<xacro:property name="visual_mesh_file" value="file://$(find py_pubsub)/models/house/myhouse.dae" />
+<xacro:property name="visual_mesh_file" value="file://$(find py_pubsub)/models/house/house.dae" />
 <link name="mapa_base">
     <visual>

Commit message: practica final ros1

File: docker_ws/py_pubsub/urdf/mapa1.xacro (robot description, xacro)
@@ -2,21 +2,21 @@
 <robot name="mapa_1" xmlns:xacro="http://www.ros.org/wiki/xacro">
 <!-- Introducir meshes -->
-<xacro:property name="visual_mesh_file" value="file://$(find py_pubsub)/models/house/house.dae" />
+<xacro:property name="visual_mesh_file" value="file://$(find py_pubsub)/models/mimundo/misilla.dae" />
 <link name="mapa_base">
     <visual>
-        <origin xyz="0 0 0" rpy="0.0 0.0 0"/>
+        <origin xyz="2 2 0" rpy="0.0 0.0 0"/>
         <geometry>
-            <mesh filename="${visual_mesh_file}" scale="1 1 1" />
+            <mesh filename="${visual_mesh_file}" scale="0.1 0.1 0.1" />
         </geometry>
     </visual>
         <!-- Se deben cambiar los parametros reales-->
     <collision>
-      <origin xyz="0 0 0" rpy="0.0 0.0 0.0"/>
+      <origin xyz="2 2 0" rpy="0.0 0.0 0.0"/>
       <geometry>
-        <mesh filename="${visual_mesh_file}" scale="1 1 1" />
+        <mesh filename="${visual_mesh_file}" scale="0.1 0.1 0.1" />
       </geometry>
     </collision>
     <inertial>
-      <origin xyz="0 0 0" rpy="0.0 0.0 0.0"/>
+      <origin xyz="2 2 0" rpy="0.0 0.0 0.0"/>
       <mass value="1"/>
       <inertia
